File: kicad/v1_4layer/ram_adapter_tsop.sch (KiCad schematic (older format))
At the start: 5 parts, among them J1 Conn_01x16_Male, J2 Conn_01x16_Male, U1 IS61C5128AL-10KLI

Commit message: Updated to 8/8 and 26/12 VIAs
Parts:
- J1: footprint Connector_PinHeader_2.54mm:PinHeader_1x16_P2.54mm_Vertical -> footprints:PinHeader_1x16_P2.54mm_Vertical
- J2: footprint Connector_PinHeader_2.54mm:PinHeader_1x16_P2.54mm_Vertical -> footprints:PinHeader_1x16_P2.54mm_VerticalAllRound
Changed lines of the file:
@@
 F 0 "J1" H 2650 2650 50  0000 C CNN
 F 1 "Conn_01x16_Male" H 2650 2750 50  0000 C CNN
-F 2 "Connector_PinHeader_2.54mm:PinHeader_1x16_P2.54mm_Vertical" H 2650 3650 50  0001 C CNN
+F 2 "footprints:PinHeader_1x16_P2.54mm_Vertical" H 2650 3650 50  0001 C CNN
 F 3 "~" H 2650 3650 50  0001 C CNN
 	1    2650 3650
@@
 F 0 "J2" H 3900 2650 50  0000 R CNN
 F 1 "Conn_01x16_Male" H 4200 2750 50  0000 R CNN
-F 2 "Connector_PinHeader_2.54mm:PinHeader_1x16_P2.54mm_Vertical" H 3850 3650 50  0001 C CNN
+F 2 "footprints:PinHeader_1x16_P2.54mm_VerticalAllRound" H 3850 3650 50  0001 C CNN
 F 3 "~" H 3850 3650 50  0001 C CNN
 	1    3850 3650
